Commit message: ROS2 warehouse robot simulation v1 (Gazebo + UR5e + control working)

File: urdf/aria_robot.urdf.xacro (robot description, xacro)
@@ -9,12 +9,14 @@
  <link name="base_link">
    <visual>
-     <geometry><box size="0.55 0.45 0.12"/></geometry>
+     <origin xyz="0 0 0.15"/>
+     <geometry><box size="0.70 0.45 0.2"/></geometry>
      <material name="navy"><color rgba="0.08 0.12 0.25 1"/></material>
    </visual>
    <collision>
-     <geometry><box size="0.55 0.45 0.12"/></geometry>
+     <origin xyz="0 0 0.15"/>
+     <geometry><box size="0.70 0.45 0.2"/></geometry>
    </collision>
    <inertial>
-     <mass value="8.0"/>
+     <mass value="40.0"/>
      <inertia ixx="0.1" ixy="0" ixz="0" iyy="0.1" iyz="0" izz="0.1"/>
    </inertial>
@@ -29,9 +31,9 @@
    <parent link="base_link"/>
    <child link="body_top"/>
-   <origin xyz="0 0 0.09"/>
+   <origin xyz="0 0 0.18"/>
  </joint>
  <link name="lidar_dome">
    <visual>
-     <geometry><cylinder radius="0.06" length="0.04"/></geometry>
+     <geometry><cylinder radius="0.06" length="0.08"/></geometry>
      <material name="white"><color rgba="0.95 0.95 0.95 1"/></material>
    </visual>
@@ -44,6 +46,6 @@
  <link name="front_bumper">
    <visual>
-     <geometry><box size="0.04 0.45 0.06"/></geometry>
-     <material name="orange"><color rgba="1.0 0.45 0.0 1"/></material>
+     <geometry><box size="0.2 0.46 0.06"/></geometry>
+     <material name="blue"><color rgba="0.6 0.8 1.0 1"/></material>
    </visual>
  </link>
@@ -51,10 +53,10 @@
    <parent link="base_link"/>
    <child link="front_bumper"/>
-   <origin xyz="0.275 0 0.0"/>
+   <origin xyz="0.275 0 0.1"/>
  </joint>
  <link name="back_bumper">
    <visual>
-     <geometry><box size="0.04 0.45 0.06"/></geometry>
-     <material name="orange"><color rgba="1.0 0.45 0.0 1"/></material>
+     <geometry><box size="0.2 0.46 0.06"/></geometry>
+     <material name="blue"><color rgba="0.6 0.8 1.0 1"/></material>
    </visual>
  </link>
@@ -62,5 +64,5 @@
    <parent link="base_link"/>
    <child link="back_bumper"/>
-   <origin xyz="-0.275 0 0.0"/>
+   <origin xyz="-0.275 0 0.1"/>
  </joint>
  <!-- ========== WHEELS ========== -->
@@ -70,14 +72,24 @@
      <material name="tire"><color rgba="0.1 0.1 0.1 1"/></material>
    </visual>
+   <collision>
+     <geometry>
+       <cylinder radius="0.09" length="0.06"/>
+     </geometry>
+  </collision>
    <inertial>
      <mass value="0.5"/>
      <inertia ixx="0.001" ixy="0" ixz="0" iyy="0.001" iyz="0" izz="0.001"/>
    </inertial>
+   <gazebo reference="front_left_wheel">
+    <mu1>5.0</mu1>
+    <mu2>5.0</mu2>
+   </gazebo>
  </link>
  <joint name="front_left_wheel_joint" type="continuous">
    <parent link="base_link"/>
    <child link="front_left_wheel"/>
-   <origin xyz="0.18 0.25 -0.04" rpy="1.5707 0 0"/>
-   <axis xyz="0 0 1"/>
+   <origin xyz="0.18 0.25 0.09" rpy="1.5707 0 0"/>
+   <axis xyz="0 0 -1"/>
+   <dynamics damping="0.2" friction="0.1"/>
  </joint>
  <link name="front_left_rim">
@@ -101,14 +113,24 @@
      <material name="tire"><color rgba="0.1 0.1 0.1 1"/></material>
    </visual>
+   <collision>
+    <geometry>
+     <cylinder radius="0.09" length="0.06"/>
+    </geometry>
+   </collision>
    <inertial>
      <mass value="0.5"/>
      <inertia ixx="0.001" ixy="0" ixz="0" iyy="0.001" iyz="0" izz="0.001"/>
    </inertial>
+   <gazebo reference="front_right_wheel">
+    <mu1>5.0</mu1>
+    <mu2>5.0</mu2>
+   </gazebo>
  </link>
  <joint name="front_right_wheel_joint" type="continuous">
    <parent link="base_link"/>
    <child link="front_right_wheel"/>
-   <origin xyz="0.18 -0.25 -0.04" rpy="1.5707 0 0"/>
-   <axis xyz="0 0 1"/>
+   <origin xyz="0.18 -0.25 0.09" rpy="1.5707 0 0"/>
+   <axis xyz="0 0 -1"/>
+   <dynamics damping="0.2" friction="0.1"/>
  </joint>
  <link name="front_right_rim">
@@ -132,14 +154,24 @@
      <material name="tire"><color rgba="0.1 0.1 0.1 1"/></material>
    </visual>
+   <collision>
+    <geometry>
+     <cylinder radius="0.09" length="0.06"/>
+    </geometry>
+   </collision>
    <inertial>
      <mass value="0.5"/>
      <inertia ixx="0.001" ixy="0" ixz="0" iyy="0.001" iyz="0" izz="0.001"/>
    </inertial>
+   <gazebo reference="back_left_wheel">
+    <mu1>5.0</mu1>
+    <mu2>5.0</mu2>
+   </gazebo>
  </link>
  <joint name="back_left_wheel_joint" type="continuous">
    <parent link="base_link"/>
    <child link="back_left_wheel"/>
-   <origin xyz="-0.18 0.25 -0.04" rpy="1.5707 0 0"/>
-   <axis xyz="0 0 1"/>
+   <origin xyz="-0.18 0.25 0.09" rpy="1.5707 0 0"/>
+   <axis xyz="0 0 -1"/>
+   <dynamics damping="0.2" friction="0.1"/>
  </joint>
  <link name="back_left_rim">
@@ -163,14 +195,24 @@
      <material name="tire"><color rgba="0.1 0.1 0.1 1"/></material>
    </visual>
+   <collision>
+    <geometry>
+     <cylinder radius="0.09" length="0.06"/>
+    </geometry>
+   </collision>
    <inertial>
      <mass value="0.5"/>
      <inertia ixx="0.001" ixy="0" ixz="0" iyy="0.001" iyz="0" izz="0.001"/>
    </inertial>
+   <gazebo reference="back_right_wheel">
+    <mu1>5.0</mu1>
+    <mu2>5.0</mu2>
+   </gazebo>
  </link>
  <joint name="back_right_wheel_joint" type="continuous">
    <parent link="base_link"/>
    <child link="back_right_wheel"/>
-   <origin xyz="-0.18 -0.25 -0.04" rpy="1.5707 0 0"/>
-   <axis xyz="0 0 1"/>
+   <origin xyz="-0.18 -0.25 0.09" rpy="1.5707 0 0"/>
+   <axis xyz="0 0 -1"/>
+   <dynamics damping="0.2" friction="0.1"/>
  </joint>
  <link name="back_right_rim">
@@ -192,6 +234,6 @@
  <link name="arm_mount">
    <visual>
-     <geometry><cylinder radius="0.08" length="0.05"/></geometry>
-     <material name="orange"><color rgba="1.0 0.45 0.0 1"/></material>
+     <geometry><cylinder radius="0.08" length="0.12"/></geometry>
+     <material name="blue"><color rgba="0.6 0.8 1.0 1"/></material>
    </visual>
  </link>
@@ -199,5 +241,5 @@
    <parent link="body_top"/>
    <child link="arm_mount"/>
-   <origin xyz="0.1 0 0.055"/>
+   <origin xyz="0.1 0 0.08"/>
  </joint>
  <!-- ========== UR5E ARM ON TOP ========== -->
@@ -210,5 +252,5 @@
    physical_parameters_file="$(find ur_description)/config/ur5e/physical_parameters.yaml"
    visual_parameters_file="$(find ur_description)/config/ur5e/visual_parameters.yaml">
-   <origin xyz="0 0 0.05" rpy="0 0 0"/>
+   <origin xyz="0 0 0.08" rpy="0 0 0"/>
  </xacro:ur_robot>
 <!-- ========== ROBOTIQ 2F-85 GRIPPER ========== -->
@@ -274,5 +316,7 @@
  <gazebo>
   <plugin filename="libgz_ros2_control-system.so"
-           name="gz_ros2_control::GazeboSimROS2ControlPlugin"/>
- </gazebo>
+          name="gz_ros2_control::GazeboSimROS2ControlPlugin">
+    <parameters>$(find warehouse_robot)/config/controllers.yaml</parameters>
+  </plugin>
+</gazebo>
 </robot>
